File: Nano_ISP_UPDI_Shield.kicad_pcb (KiCad board)
At the start: 2 copper layers, 18.3 x 46.2 mm, 5 parts, among them J1 UPDI, J2 pwrselect

Commit message: version1
Parts:
- J2: moved to B.Cu
- turned J2 to 0 degrees
Other:
- board text added: "Pwr Sel UPDI Only"
